File: SBCBufferedLink.kicad_sch (KiCad schematic)
At the start: 9 parts, among them J2 Left, J2 Right

Commit message: add board edge
Other:
- title: (none) -> HD6309 SBC Backplane Link
Changed lines of the file:
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@@
 (kicad_sch (version 20230121) (generator eeschema)
   (paper "A4")
+  (title_block
+    (title "HD6309 SBC Backplane Link")
+    (date "2023-04-24")
+    (rev "Revision 1")
+  )
   (no_connect (at 34.3916 20.5232))
   (no_connect (at 245.8466 28.1178))

Commit message: complete tracing
Connections:
- net A10: now also U6.15 (B4)
- net A10_LEFT: now also U6.6 (A4)
- net A11: now also U6.13 (B6)
- net A11_LEFT: now also U6.8 (A6)
- net A12: now also U6.11 (B8)
- net A12_LEFT: now also U6.10 (A8)
- net A13: now also U3.17 (B2)
- net A13_LEFT: now also U3.4 (A2)
- net A14: now also U3.15 (B4)
- net A14_LEFT: now also U3.6 (A4)
- net A15: now also U3.13 (B6)
- net A15_LEFT: now also U3.8 (A6)
- net A5: now also U2.17 (B2)
- net A5_LEFT: now also U2.4 (A2)
- net A6: now also U2.15 (B4)
- net A6_LEFT: now also U2.6 (A4)
- net A7: now also U2.13 (B6)
- net A7_LEFT: now also U2.8 (A6)
- net A8: now also U2.11 (B8)
- net A8_LEFT: now also U2.10 (A8)
- net A9: now also U6.17 (B2)
- net A9_LEFT: now also U6.4 (A2)
- net BA: now also U4.17 (B2)
- net BA_LEFT: now also U4.4 (A2)
- net BS: now also U4.15 (B4)
- net BS_LEFT: now also U4.6 (A4)
- net D4: now also U2.18 (B1)
- net D4_LEFT: now also U2.3 (A1)
- net D5: now also U2.16 (B3)
- net D5_LEFT: now also U2.5 (A3)
- net D6: now also U2.14 (B5)
- net D6_LEFT: now also U2.7 (A5)
- net D7: now also U2.12 (B7)
- net D7_LEFT: now also U2.9 (A7)
- net MAPPED_MEM: now also U6.18 (B1)
- net MAPPED_MEM_LEFT: now also U6.3 (A1)
- net MRDY: now also U4.14 (B5)
- net MRDY_LEFT: now also U4.7 (A5)
- net Q1: now also U6.14 (B5)
- net Q1_LEFT: now also U6.7 (A5)
- net Q2: now also U6.12 (B7)
- net Q2_LEFT: now also U6.9 (A7)
- net Q3: now also U3.18 (B1)
- net Q3_LEFT: now also U3.3 (A1)
- net Q4: now also U3.16 (B3)
- net Q4_LEFT: now also U3.5 (A3)
- net Q5: now also U3.14 (B5)
- net Q5_LEFT: now also U3.7 (A5)
- net Q6: now also U3.12 (B7)
- net Q6_LEFT: now also U3.9 (A7)
- net Q7: now also U8.18 (B1)
- net Q7_LEFT: now also U8.3 (A1)
- net Q8: now also U8.16 (B3)
- net Q8_LEFT: now also U8.5 (A3)
- net ROM/~{RAM}: now also U6.16 (B3)
- net ROM/~{RAM}_LEFT: now also U6.5 (A3)
- net R/~{W}: now also U8.12 (B7)
- net R/~{W}_LEFT: now also U8.9 (A7)
- net ~{DMA}: now also U8.14 (B5)
- net ~{DMA}_LEFT: now also U8.7 (A5)
- net ~{FIRQ}: now also U8.13 (B6)
- net ~{FIRQ}_LEFT: now also U8.8 (A6)
- net ~{HALT}: now also U4.18 (B1)
- net ~{HALT}_LEFT: now also U4.3 (A1)
- net ~{IRQ}: now also U8.11 (B8)
- net ~{IRQ}_LEFT: now also U8.10 (A8)
- net ~{NMI}: now also U8.15 (B4)
- net ~{NMI}_LEFT: now also U8.6 (A4)
- net ~{RESET}: now also U8.17 (B2)
- net ~{RESET}_LEFT: now also U8.4 (A2)
- net NC5_LEFT: now reaches U4.10 (A8)
- net NC5_LEFT: now also J2.59 (Pin_59)
- net NC5: now reaches U4.11 (B8)
- net NC5: now also J2.59 (Pin_59)
- net NC3: now reaches U4.12 (B7)
- net NC3: now also J2.57 (Pin_57)
- net NC4: now reaches U4.13 (B6)
- net NC4: now also J2.58 (Pin_58)
- net NC2: now reaches U4.16 (B3)
- net NC2: now also J2.53 (Pin_53)
- net NC2_LEFT: now reaches U4.5 (A3)
- net NC2_LEFT: now also J2.53 (Pin_53)
- net NC4_LEFT: now reaches U4.8 (A6)
- net NC4_LEFT: now also J2.58 (Pin_58)
- net NC3_LEFT: now reaches U4.9 (A7)
- net NC3_LEFT: now also J2.57 (Pin_57)
- net NC1_LEFT: now reaches U3.10 (A8)
- net NC1_LEFT: now also J2.44 (Pin_44)
- net NC1: now reaches U3.11 (B8)
- net NC1: now also J2.44 (Pin_44)
- no-connect marks 14 -> 4
